File: Serial-Ethernet-HW.kicad_pcb (KiCad board)
At the start: 4 copper layers, 41.1 x 50.7 mm, 52 parts, among them J1 7499111121A, J2 UJ2-MBH-1-SMT-TR, J3 D09P33E4GX00LF, U1 W5500, U2 MPM3612-33, U3 STM32G061GxUx, Y1 ECS-250-10-37B-CTN-TR

Commit message: Rebuild using new output scripts
Parts:
- moved C1 150.7 mm to (80.0, 80.3)
- moved C10 150.7 mm to (75.2, 85.5)
- moved C11 150.7 mm to (76.7, 85.5)
- moved C12 150.7 mm to (66.6, 85.6)
- moved C13 150.7 mm to (60.2, 81.9)
- moved C14 150.7 mm to (58.6, 78.9)
- moved C15 150.7 mm to (58.6, 77.4)
- moved C16 150.7 mm to (60.1, 72.8)
- moved C17 150.7 mm to (84.4, 61.9)
- moved C18 150.7 mm to (82.6, 61.9)
- moved C19 150.7 mm to (83.1, 68.7)
- moved C2 150.7 mm to (82.3, 79.4)
- moved C20 150.7 mm to (77.5, 61.8)
- moved C21 150.7 mm to (81.6, 68.7)
- moved C22 150.7 mm to (75.7, 61.9)
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Connections:
- net /Ethernet/3V3A renamed +3V3A
- J1 pad 10: unconnected-(J1-Pad10) -> GND
Other:
- board text added: "Serial to Ethernet v1.0b Sep 25"
- board text removed: "Serial to Ethernet v1.0 Feb 23"
