File: Serial-Ethernet-HW.kicad_sch (KiCad schematic)
At the start: 0 parts

Commit message: Rebuild using new output scripts
Other:
- company: (none) -> TL Embedded Ltd
- title: (none) -> Serial-Ethernet
