File: Ethernet.kicad_sch (KiCad schematic)
At the start: 30 parts, among them J1 7499111121A, U1 W5500, Y1 ECS-250-10-37B-CTN-TR

Commit message: Add in RS232
Parts:
- removed C12: 10u, C_Capacitor:C_0805, symbol C_Capacitor:C_0805
- removed C9: 4u7, C_Capacitor:C_0603, symbol C_Capacitor:C_0603
- removed L1: 600R, L_Inductor:FB_0603, symbol L_Inductor:FB_0603
- added C12, C8: 4u7,10v, C_Capacitor:C_0603, symbol C_Capacitor:C_0603
- added L1: BLM18KG601SN1D, L_Inductor:FB_0603, symbol L_Inductor:BLM18KG601SN1D
- R10, R9: value 330R -> 470R
- renumbered C2 to C1, C3 to C2, C1 to C3, C8 to C9
Connections:
- net +3V3: now also L1.1
- net +3V3A: now also C12.1, L1.2
- net GND: now also C12.2, C8.2
- net at U1.20 (TOCAP): now also C8.1
Other:
- company: TL Embedded Ltd -> TL Embedded
- moved on the sheet: R2
